File: hardware/imu_to_dxl/imu_to_dxl.kicad_sch (KiCad schematic)
At the start: 74 parts, among them J1 1.8mm螺丝孔, J2 1.8mm螺丝孔, J3 1.8mm螺丝孔, J4 1.8mm螺丝孔, Q1 MMBT3906, U1 ETA2845S2G_C22362741, U2 GD32F303CCT6, U3 LSM6DSV16XTR, U4 SN74LVC1G126DBVR, U5 SN74LVC1G125DBV, U6 ME6211C18M5G-N, X1 XL2EL89CSI-111YLC-12M

Commit message: 修改IMU工作电压到5V；拼板文件优化
Parts:
- R4: now not fitted; now left out of the parts list
Other:
- note removed: "UVLO=3V"
Changed lines of the file:
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@@
 	(generator_version "9.0")
 	(paper "A3")
-	(text "UVLO=3V"
-		(exclude_from_sim no)
-		(at 217.17 44.704 0)
-		(effects
-			(font
-				(size 1.27 1.27)
-			)
-		)
-	)
 	(text "Debug"
 		(exclude_from_sim no)
@@
 		(unit 1)
 		(exclude_from_sim no)
-		(in_bom yes)
+		(in_bom no)
 		(on_board yes)
-		(dnp no)
+		(dnp yes)
 		(fields_autoplaced yes)
 		(property "Reference" "R4"

Commit message: 更新imu_to_dxl:1、优化MCU晶震电路；2、增加调试知识灯
Parts:
- added LED1: GL0603UG01, microduck:LED0603-RD, symbol microduck:GL0603UG01
- added R34: 100K, microduck:R0402, symbol microduck:RC0402FR-0710KL
- added R35: 1M, microduck:R0402, symbol microduck:RC0402FR-0710KL
- C10, C11: value 27pF/50V -> 20pF/50V; LCSC Part C107002 -> C107000
- CN1: value ~ -> B3B-EH-A(LF)(SN)
- CN2: value ~ -> AMP175778/8283/A2007WV-3P
- D1: value SMAJ24A -> SMAJ36A; LCSC Part C90510 -> C353452; Manufacturer Brightking(君耀电子) -> (none); Manufacturer Part SMAJ24A/TR13 -> (none)
- R5: value 51R -> 0R; LCSC Part C2907181 -> C21189
Connections:
- net GD_OSCIN: now also R35.2
- net GD_OSCOUT: now also R35.1
- net GND: now also R34.2
- net DEBUG_LED: now reaches U2.41 (PB5)
- net DEBUG_LED: now also LED1.2 (A)
- new net: LED1.1 (K), R34.1
Other:
- note removed: "改6.3V"
